File: Controlador-Compressor/Controlador-Compressor.kicad_pcb (KiCad board)
At the start: 2 copper layers, 24.5 x 33.8 mm, 85 parts, among them J1 RELÉ-1, J2 RELÉ-2, J3 RELÉ-3, J4 RELÉ-4, J5 RELÉ-5, J6 Analogico, J7 Alimentação, J8 modbus, K1 FINDER-36.11, K2 FINDER-36.11, K3 FINDER-36.11, K4 FINDER-36.11, K5 FINDER-36.11, Q1 BC817, Q2 BC817, U1 ESP32S3WROOM1N8R8, U10 CP2102N-Axx-xQFN28, U2 PC817, U3 PC817, U4 PC817, U5 PC817, U6 PC817, U7 LM358, U8 AMS1117-3.3, U9 SN75176ADR

Commit message: mei caminho andado
Parts:
- removed C19, C21, C22: 220nF, Capacitor_SMD:C_0402_1005Metric
- removed C20: 1.5pF, Capacitor_SMD:C_0402_1005Metric
- removed C23, C24: 10uF, Capacitor_SMD:C_0603_1608Metric
- removed D16: SRV05-4-P-T7, Package_TO_SOT_SMD:SOT-23-6
- removed R18, R19, R29, R30: 5.1K, Resistor_SMD:R_0402_1005Metric
- removed R27, R28: 100k, Resistor_SMD:R_0402_1005Metric
- removed U10: CP2102N-Axx-xQFN28, Package_DFN_QFN:QFN-28-1EP_5x5mm_P0.5mm_EP3.35x3.35mm
- added C17: 10uF, Capacitor_SMD:C_0603_1608Metric, F.Cu at (264.6, 65.5)
- added C4: 1.5pF, Capacitor_SMD:C_0402_1005Metric, F.Cu at (261.1, 38.9)
- added C5: 1.5pF, Capacitor_SMD:C_0402_1005Metric, F.Cu at (261.1, 40.9)
- added C6: 220nF, Capacitor_SMD:C_0402_1005Metric, F.Cu at (261.1, 42.8)
- added C7: 220nF, Capacitor_SMD:C_0402_1005Metric, F.Cu at (261.1, 44.8)
- added C8: 1.5pF, Capacitor_SMD:C_0402_1005Metric, F.Cu at (261.1, 46.8)
- added D15: SRV05-4-P-T7, Package_TO_SOT_SMD:SOT-23-6, F.Cu at (265.1, 54.4)
- added Q3: BC817, Package_TO_SOT_SMD:SOT-23, F.Cu at (228.1, 103.4)
- added R10: 100k, Resistor_SMD:R_0402_1005Metric, F.Cu at (261.1, 48.8)
- added R11: 100k, Resistor_SMD:R_0402_1005Metric, F.Cu at (261.1, 50.8)
- added R12: 100k, Resistor_SMD:R_0402_1005Metric, F.Cu at (261.1, 52.7)
- added R13: 100k, Resistor_SMD:R_0402_1005Metric, F.Cu at (261.1, 54.7)
- added R14: 5.1K, Resistor_SMD:R_0402_1005Metric, F.Cu at (261.1, 56.7)
- added R15: 5.1K, Resistor_SMD:R_0402_1005Metric, F.Cu at (261.1, 58.7)
- added R35: 1k, Resistor_SMD:R_0603_1608Metric_Pad0.98x0.95mm_HandSolder, F.Cu at (232.6, 99.8)
- C11: value 1.5pF -> 220nF
- C16: footprint Capacitor_SMD:C_0603_1608Metric_Pad1.08x0.95mm_HandSolder -> Capacitor_SMD:C_0603_1608Metric
- C18: value 1.5pF -> 10uF; footprint Capacitor_SMD:C_0402_1005Metric -> Capacitor_SMD:C_0603_1608Metric_Pad1.08x0.95mm_HandSolder
- D10: value D -> LED; footprint Diode_THT:D_A-405_P2.54mm_Vertical_KathodeUp -> LED_SMD:LED_0805_2012Metric_Pad1.15x1.40mm_HandSolder
- D5: value LED -> D; footprint LED_SMD:LED_0805_2012Metric_Pad1.15x1.40mm_HandSolder -> Diode_THT:D_A-405_P2.54mm_Vertical_KathodeUp
- R16, R17: value 100k -> 5.1K
- R31: value 100k -> 33k
- R33: value 33k -> 100k
- U1: value ESP32S3WROOM1N8R8 -> CP2102N-Axx-xQFN28; footprint esp32s3:XCVR_ESP32S3WROOM1N8R8 -> Package_DFN_QFN:QFN-28-1EP_5x5mm_P0.5mm_EP3.35x3.35mm
- U6: value PC817 -> ESP32S3WROOM1N8R8; footprint Package_DIP:DIP-4_W7.62mm -> esp32s3:XCVR_ESP32S3WROOM1N8R8
- moved U1 119.5 mm to (269.0, 41.5)
- moved C10 110.9 mm to (264.0, 40.9)
- moved C11 110.9 mm to (264.0, 42.8)
- moved C12 110.9 mm to (264.0, 44.8)
- moved C13 110.9 mm to (264.0, 46.8)
- moved C9 110.9 mm to (264.0, 38.9)
- moved C18 104.9 mm to (267.6, 46.4)
- moved Q1 102.3 mm to (270.2, 50.0)
- moved Q2 102.3 mm to (270.2, 54.4)
- moved J6 84.4 mm to (247.8, 74.1)
- moved R17 80.3 mm to (261.1, 62.7)
- moved R16 80.3 mm to (261.1, 60.7)
- moved U6 80.0 mm to (294.1, 55.4)
- moved FL1 80.0 mm to (268.3, 63.8)
- moved FL2 80.0 mm to (268.3, 67.0)
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Connections:
- net /0_10V_MCU1 renamed /Analógico/0_10V_MCU1
- net /0_10V_MCU2 renamed /Analógico/0_10V_MCU2
- C10 pad 1: /VBUS_5V -> VBUS
- C11 pad 1: GND -> VBUS
- C11 pad 2: Net-(C11-Pad2) -> GND
- C16 pad 1: +3V3 -> VBUS
- C18 pad 1: GND -> +3V3
- C18 pad 2: Net-(C18-Pad2) -> GND
- D1 pad 2: /RELÉ-1 -> /Potência/RELÉ-2
- D10 pad 1: +24V -> Net-(D10-K)
- D14 pad 1: /SHIELD -> /ESP32-S3/ESP_SHIELD
- D14 pad 4: /D- -> /ESP32-S3/ESP_D-
- D14 pad 5: /VBUS_5V -> /ESP32-S3/VBUS_5V
- D14 pad 6: /D+ -> /ESP32-S3/ESP_D+
- D2 pad 2: /RELÉ-2 -> /Potência/RELÉ-3
- D3 pad 2: /RELÉ-3 -> /Potência/RELÉ-4
- D4 pad 2: /RELÉ-4 -> /Potência/RELÉ-5
- D5 pad 1: Net-(D5-K) -> +24V
- D5 pad 2: /RELÉ-5 -> Net-(D10-A)
- FL1 pad 1: /D+ -> /ESP32-S3/D+
- FL1 pad 2: /D- -> /ESP32-S3/D-
- FL1 pad 5: /USB_D- -> /ESP32-S3/USB_D-
- FL1 pad 6: /USB_D+ -> /ESP32-S3/USB_D+
- FL2 pad 1: /ESP_D+ -> /ESP32-S3/ESP_D+
- FL2 pad 2: /ESP_D- -> /ESP32-S3/ESP_D-
- FL2 pad 5: /GPIO19 -> /ESP32-S3/GPIO19
- FL2 pad 6: /GPIO20 -> /ESP32-S3/GPIO20
- J6 pad 1: /0_10V_OUT1 -> /Analógico/0_10V_OUT1
- J6 pad 2: /0_10V_OUT2 -> /Analógico/0_10V_OUT2
- K1 pad A2: Net-(D6-A) -> Net-(D10-A)
- K2 pad A2: Net-(D7-A) -> Net-(D6-A)
- K3 pad A2: Net-(D8-A) -> Net-(D7-A)
- K4 pad A2: Net-(D9-A) -> Net-(D8-A)
- K5 pad A2: Net-(D10-A) -> Net-(D9-A)
- L1 pad 1: /VBUS_5V -> /ESP32-S3/VBUS_5V
- L2 pad 1: /ESP_VBUS_5V -> /ESP32-S3/ESP_VBUS_5V
- Q1 pad 2: /RTS -> /ESP32-S3/RTS
- Q2 pad 2: /DTR -> /ESP32-S3/DTR
- R16 pad 1: Net-(C9-Pad2) -> /ESP32-S3/ESP_CC1
- R16 pad 2: /SHIELD -> GND
- R17 pad 1: Net-(C11-Pad2) -> /ESP32-S3/CC1
- R17 pad 2: /SHIELD -> GND
- R31 pad 1: GND -> /Analógico/0_10V_OUT1
- R31 pad 2: /0_10V_FB_1 -> /Analógico/0_10V_FB_1
- R32 pad 1: /0_10V_OUT1 -> /Analógico/0_10V_OUT2
- R32 pad 2: /0_10V_FB_1 -> /Analógico/0_10V_FB_2
- R33 pad 1: /0_10V_OUT2 -> GND
- R33 pad 2: /0_10V_FB_2 -> /Analógico/0_10V_FB_1
- R34 pad 2: /0_10V_FB_2 -> /Analógico/0_10V_FB_2
- R5 pad 1: Net-(D5-K) -> /Potência/RELÉ-1
- R5 pad 2: Net-(R5-Pad2) -> Net-(Q3-B)
- U1 pad 1: GND -> unconnected-(U1-~{DCD}-Pad1)
- U1 pad 10: /DE -> unconnected-(U1-NC-Pad10)
- U1 pad 11: /RS485_TX -> Net-(U1-~{SUSPEND})
- U1 pad 12: /RELÉ-5 -> unconnected-(U1-SUSPEND-Pad12)
- U1 pad 13: /GPIO19 -> unconnected-(U1-CHREN-Pad13)
- U1 pad 14: /GPIO20 -> unconnected-(U1-CHR1-Pad14)
- U1 pad 15: /GPIO3 -> unconnected-(U1-CHR0-Pad15)
- U1 pad 16: Net-(U1-IO46) -> unconnected-(U1-~{WAKEUP}/GPIO.3-Pad16)
- U1 pad 2: +3V3 -> unconnected-(U1-~{RI}/CLK-Pad2)
- U1 pad 23: /~{RE} -> unconnected-(U1-~{CTS}-Pad23)
- U1 pad 24: unconnected-(U1-IO47-Pad24) -> /ESP32-S3/RTS
- U1 pad 25: unconnected-(U1-IO48-Pad25) -> /ESP32-S3/TXD0
- U1 pad 26: Net-(U1-IO45) -> /ESP32-S3/RXD0
- U1 pad 27: /GPIO0 -> unconnected-(U1-~{DSR}-Pad27)
- U1 pad 28: /RS485_RX -> /ESP32-S3/DTR
- U1 pad 29: unconnected-(U1-IO36-Pad29) -> GND
- U1 pad 3: /RST -> GND
- U1 pad 4: /RELÉ-1 -> /ESP32-S3/USB_D+
- U1 pad 5: /RELÉ-2 -> /ESP32-S3/USB_D-
- U1 pad 6: /RELÉ-3 -> +3V3
- U1 pad 7: /RELÉ-4 -> +3V3
- U1 pad 8: unconnected-(U1-IO15-Pad8) -> Net-(U1-VBUS)
- U1 pad 9: unconnected-(U1-IO16-Pad9) -> Net-(U1-~{RST})
- U6 pad 1: Net-(R5-Pad2) -> GND
- U6 pad 2: GND -> +3V3
- U6 pad 3: GND -> /ESP32-S3/RST
- U6 pad 4: Net-(D10-A) -> /ESP32-S3/RELÉ-1

Commit message: terminei escopo do projeto
Parts:
- removed D13: WS2812B, LED_SMD:LED_WS2812B_PLCC4_5.0x5.0mm_P3.2mm
- removed D9: D, Diode_THT:D_A-405_P2.54mm_Vertical_KathodeUp
- removed IN+1: IN+, Connector_PinHeader_2.54mm:PinHeader_1x01_P2.54mm_Vertical
- removed IN-1: IN-, Connector_PinHeader_2.54mm:PinHeader_1x01_P2.54mm_Vertical
- removed J1: RELÉ-1, Connector_Phoenix_MSTB:PhoenixContact_MSTBA_2,5_3-G-5,08_1x03_P5.08mm_Horizontal
- removed J2: RELÉ-2, Connector_Phoenix_MSTB:PhoenixContact_MSTBA_2,5_3-G-5,08_1x03_P5.08mm_Horizontal
- removed J3: RELÉ-3, Connector_Phoenix_MSTB:PhoenixContact_MSTBA_2,5_3-G-5,08_1x03_P5.08mm_Horizontal
- removed J4: RELÉ-4, Connector_Phoenix_MSTB:PhoenixContact_MSTBA_2,5_3-G-5,08_1x03_P5.08mm_Horizontal
- removed J5: RELÉ-5, Connector_Phoenix_MSTB:PhoenixContact_MSTBA_2,5_3-G-5,08_1x03_P5.08mm_Horizontal
- removed J8: modbus, Connector_Phoenix_MSTB:PhoenixContact_MSTBA_2,5_3-G-5,08_1x03_P5.08mm_Horizontal
- removed OUT+1: OUT+, Connector_PinHeader_2.54mm:PinHeader_1x01_P2.54mm_Vertical
- removed OUT-1: OUT-, Connector_PinHeader_2.54mm:PinHeader_1x01_P2.54mm_Vertical
- added D19: LED, LED_SMD:LED_0805_2012Metric_Pad1.15x1.40mm_HandSolder, F.Cu at (303.7, 85.7)
- added D20: WS2812B, LED_SMD:LED_WS2812B_PLCC4_5.0x5.0mm_P3.2mm, F.Cu at (333.9, 163.1)
- added D21: D, Diode_THT:D_A-405_P2.54mm_Vertical_KathodeUp, F.Cu at (296.6, 94.2)
- added D22: LED, LED_SMD:LED_0805_2012Metric_Pad1.15x1.40mm_HandSolder, F.Cu at (303.7, 88.7)
- added J11: Saídas Relé, Connector_Phoenix_MSTB:PhoenixContact_MSTBA_2,5_12-G-5,08_1x12_P5.08mm_Horizontal, F.Cu at (135.1, 126.5)
- added J13: Analógico, Connector_Phoenix_MSTB:PhoenixContact_MSTBA_2,5_16-G-5,08_1x16_P5.08mm_Horizontal, F.Cu at (135.1, 112.0)
- added J16: Nextion, Connector_JST:JST_EH_B4B-EH-A_1x04_P2.50mm_Vertical, F.Cu at (199.1, 125.7)
- added K6: FINDER-36.11, Relay_THT:Relay_SPDT_Finder_36.11, F.Cu at (276.6, 133.7)
- added Q4: BC817, Package_TO_SOT_SMD:SOT-23, F.Cu at (297.4, 102.8)
- added Q5: BC817, Package_TO_SOT_SMD:SOT-23, F.Cu at (297.4, 107.2)
- added Q6: BC817, Package_TO_SOT_SMD:SOT-23, F.Cu at (297.4, 111.7)
- added Q7: BC817, Package_TO_SOT_SMD:SOT-23, F.Cu at (297.4, 116.1)
- added Q8: BC817, Package_TO_SOT_SMD:SOT-23, F.Cu at (302.3, 102.8)
- added R36: 1k, Resistor_SMD:R_0603_1608Metric_Pad0.98x0.95mm_HandSolder, F.Cu at (297.1, 129.7)
- added R37: 1k, Resistor_SMD:R_0603_1608Metric_Pad0.98x0.95mm_HandSolder, F.Cu at (301.5, 119.6)
- added R38: 1k, Resistor_SMD:R_0603_1608Metric_Pad0.98x0.95mm_HandSolder, F.Cu at (301.5, 122.1)
- added R39: 1k, Resistor_SMD:R_0603_1608Metric_Pad0.98x0.95mm_HandSolder, F.Cu at (301.5, 124.6)
- added R42: 1k, Resistor_SMD:R_0603_1608Metric_Pad0.98x0.95mm_HandSolder, F.Cu at (301.5, 127.2)
- added R43: 1k, Resistor_SMD:R_0603_1608Metric_Pad0.98x0.95mm_HandSolder, F.Cu at (301.5, 129.7)
- added U10: PC817, Package_DIP:DIP-4_W7.62mm, F.Cu at (132.2, 161.7)
- added U11: PC817, Package_DIP:DIP-4_W7.62mm, F.Cu at (132.2, 168.4)
- D1, D3: value LED -> D; footprint LED_SMD:LED_0805_2012Metric_Pad1.15x1.40mm_HandSolder -> Diode_THT:D_A-405_P2.54mm_Vertical_KathodeUp
- D8: value D -> LED; footprint Diode_THT:D_A-405_P2.54mm_Vertical_KathodeUp -> LED_SMD:LED_0805_2012Metric_Pad1.15x1.40mm_HandSolder
- U2: value PC817 -> LM2596S-5; footprint Package_DIP:DIP-4_W7.62mm -> Package_TO_SOT_SMD:TO-263-5_TabPin3
- U3: value PC817 -> SN75176ADR; footprint Package_DIP:DIP-4_W7.62mm -> Package_SO:SOIC-8_3.9x4.9mm_P1.27mm
- U9: value SN75176ADR -> PC817; footprint Package_SO:SOIC-8_3.9x4.9mm_P1.27mm -> Package_DIP:DIP-4_W7.62mm
- moved C9 171.1 mm to (151.7, 168.0)
- moved C11 169.6 mm to (151.7, 170.0)
- moved C13 168.1 mm to (151.7, 172.0)
- moved C5 164.7 mm to (151.7, 164.1)
- moved C7 163.3 mm to (151.7, 166.0)
- moved D14 162.8 mm to (146.0, 160.9)
- moved C10 160.6 mm to (149.7, 153.7)
- moved FL2 160.4 mm to (145.1, 169.7)
- moved R11 159.5 mm to (148.9, 164.1)
- moved C12 159.2 mm to (149.7, 155.7)
- moved Q1 158.9 mm to (145.8, 149.0)
- moved Q2 158.9 mm to (145.8, 153.5)
- moved U1 158.8 mm to (147.0, 143.2)
- moved C15 158.1 mm to (145.4, 164.3)
- moved R13 158.1 mm to (148.9, 166.1)
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Connections:
- net /Analógico/0_10V_FB_1 renamed /Circuito Analógico/0_10V_FB_1
- net /Analógico/0_10V_FB_2 renamed /Circuito Analógico/0_10V_FB_2
- net /Analógico/0_10V_MCU1 renamed /Circuito Analógico/0_10V_MCU1
- net /Analógico/0_10V_MCU2 renamed /Circuito Analógico/0_10V_MCU2
- net /Analógico/0_10V_OUT1 renamed /Circuito Analógico/0_10V_OUT1
- net /Analógico/0_10V_OUT2 renamed /Circuito Analógico/0_10V_OUT2
- net /ESP32-S3/CC1 renamed /USB->UART/CC1
- net /ESP32-S3/CC2 renamed /USB->UART/CC2
- net /ESP32-S3/D+ renamed /USB->UART/D+
- net /ESP32-S3/D- renamed /USB->UART/D-
- net /ESP32-S3/DTR renamed /USB->UART/DTR
- net /ESP32-S3/ESP_CC1 renamed /USB->OTG/ESP_CC1
- net /ESP32-S3/ESP_CC2 renamed /USB->OTG/ESP_CC2
- net /ESP32-S3/ESP_D+ renamed /USB->OTG/ESP_D+
- net /ESP32-S3/ESP_D- renamed /USB->OTG/ESP_D-
- net /ESP32-S3/ESP_SHIELD renamed /USB->OTG/ESP_SHIELD
- net /ESP32-S3/ESP_VBUS_5V renamed /USB->OTG/ESP_VBUS_5V
- net /ESP32-S3/GPIO19 renamed /USB->OTG/GPIO19
- net /ESP32-S3/GPIO20 renamed /USB->OTG/GPIO20
- net /ESP32-S3/RELÉ-1 renamed /Circuito Analógico/MCU-AI3
- net /ESP32-S3/RELÉ-2 renamed /Circuito Analógico/MCU-AI4
- net /ESP32-S3/RELÉ-3 renamed /Circuito Analógico/MCU-AI5
- net /ESP32-S3/RELÉ-4 renamed /Circuito Analógico/MCU-AI6
- net /ESP32-S3/RELÉ-5 renamed /Circuito Analógico/MCU-AI7
- net /ESP32-S3/RTS renamed /USB->UART/RTS
- net /ESP32-S3/SHIELD renamed /USB->UART/SHIELD
- net /ESP32-S3/USB_D+ renamed /USB->UART/USB_D+
- net /ESP32-S3/USB_D- renamed /USB->UART/USB_D-
- net /RS485_RX renamed Net-(R50-Pad1)
- C6 pad 1: /ESP32-S3/VBUS_5V -> /USB->UART/VBUS_5V
- D1 pad 1: Net-(D1-K) -> +24V
- D1 pad 2: /Potência/RELÉ-2 -> Net-(D1-A)
- D14 pad 5: /ESP32-S3/VBUS_5V -> /USB->OTG/VBUS_5V
- D15 pad 5: /ESP32-S3/VBUS_5V -> /USB->UART/VBUS_5V
- D2 pad 2: /Potência/RELÉ-3 -> Net-(D1-A)
- D3 pad 1: Net-(D3-K) -> +24V
- D3 pad 2: /Potência/RELÉ-4 -> Net-(D3-A)
- D4 pad 2: /Potência/RELÉ-5 -> Net-(D3-A)
- D6 pad 2: Net-(D6-A) -> Net-(D19-A)
- D8 pad 1: +24V -> Net-(D8-K)
- D8 pad 2: Net-(D8-A) -> Net-(D7-A)
- K1 pad 11: Net-(J1-Pin_2) -> /Circuito digital/COM0
- K1 pad 12: Net-(J1-Pin_3) -> unconnected-(K1-Pad12)
- K1 pad 14: Net-(J1-Pin_1) -> /Circuito digital/DO0
- K2 pad 11: Net-(J2-Pin_2) -> /Circuito digital/COM1
- K2 pad 12: Net-(J2-Pin_3) -> unconnected-(K2-Pad12)
- K2 pad 14: Net-(J2-Pin_1) -> /Circuito digital/DO1
- K2 pad A2: Net-(D6-A) -> Net-(D19-A)
- K3 pad 11: Net-(J3-Pin_2) -> /Circuito digital/COM2
- K3 pad 12: Net-(J3-Pin_3) -> unconnected-(K3-Pad12)
- K3 pad 14: Net-(J3-Pin_1) -> /Circuito digital/DO2
- K3 pad A2: Net-(D7-A) -> Net-(D1-A)
- K4 pad 11: Net-(J4-Pin_2) -> /Circuito digital/COM3
- K4 pad 12: Net-(J4-Pin_3) -> unconnected-(K4-Pad12)
- K4 pad 14: Net-(J4-Pin_1) -> /Circuito digital/DO3
- K4 pad A2: Net-(D8-A) -> Net-(D3-A)
- K5 pad 11: Net-(J5-Pin_2) -> /Circuito digital/COM4
- K5 pad 12: Net-(J5-Pin_3) -> unconnected-(K5-Pad12)
- K5 pad 14: Net-(J5-Pin_1) -> /Circuito digital/DO4
- K5 pad A2: Net-(D9-A) -> Net-(D7-A)
- L1 pad 1: /ESP32-S3/VBUS_5V -> /USB->UART/VBUS_5V
- Q3 pad 3: Net-(D10-K) -> Net-(Q3-C)
- R1 pad 1: Net-(D1-K) -> Net-(Q4-B)
- R1 pad 2: Net-(R1-Pad2) -> /Circuito digital/RELE 2
- R2 pad 1: Net-(D2-K) -> /Circuito digital/RELE 3
- R2 pad 2: Net-(R2-Pad2) -> Net-(Q5-B)
- R3 pad 1: Net-(D3-K) -> Net-(Q5-C)
- R3 pad 2: Net-(R3-Pad2) -> Net-(D2-K)
- R35 pad 1: unconnected-(R35-Pad1) -> Net-(Q3-C)
- R35 pad 2: unconnected-(R35-Pad2) -> Net-(D10-K)
- R4 pad 1: Net-(D4-K) -> /Circuito digital/RELE 4
- R4 pad 2: Net-(R4-Pad2) -> Net-(Q6-B)
- R5 pad 1: /Potência/RELÉ-1 -> /Circuito digital/RELE 1
- U1 pad 25: /ESP32-S3/TXD0 -> /ESP32-S3/RXD0
- U1 pad 26: /ESP32-S3/RXD0 -> /ESP32-S3/TXD0
- U2 pad 1: Net-(R1-Pad2) -> +24V
- U2 pad 2: GND -> Net-(D18-K)
- U2 pad 4: Net-(D6-A) -> Net-(U2-FB)
- U3 pad 1: Net-(R2-Pad2) -> /ESP32-S3/RS485_RX
- U3 pad 2: GND -> /ESP32-S3/DE
- U3 pad 3: GND -> /ESP32-S3/DE
- U3 pad 4: Net-(D7-A) -> /ESP32-S3/RS485_TX
- U4 pad 1: Net-(R3-Pad2) -> Net-(R45-Pad1)
- U4 pad 4: Net-(D8-A) -> /Circuito digital/DI0
- U5 pad 1: Net-(R4-Pad2) -> Net-(R48-Pad1)
- U5 pad 4: Net-(D9-A) -> /Circuito digital/DI1
- U6 pad 10: /ESP32-S3/DE -> /ESP32-S3/RX-Nextion
- U6 pad 11: /ESP32-S3/RS485_TX -> /ESP32-S3/Tx-Nextion
- U6 pad 17: unconnected-(U6-IO9-Pad17) -> /Circuito Analógico/MCU-AI8
- U6 pad 18: unconnected-(U6-IO10-Pad18) -> /Circuito Analógico/MCU-AI9
- U6 pad 19: unconnected-(U6-IO11-Pad19) -> /Circuito digital/RELE 1
- U6 pad 20: unconnected-(U6-IO12-Pad20) -> /Circuito digital/RELE 2
- U6 pad 21: unconnected-(U6-IO13-Pad21) -> /Circuito digital/RELE 3
- U6 pad 22: unconnected-(U6-IO14-Pad22) -> /Circuito digital/RELE 4
- U6 pad 23: /ESP32-S3/~{RE} -> /ESP32-S3/RS485_RX
- U6 pad 24: unconnected-(U6-IO47-Pad24) -> /Circuito digital/DI3
- U6 pad 25: unconnected-(U6-IO48-Pad25) -> /Circuito digital/DI4
- U6 pad 28: /ESP32-S3/RS485_RX -> /ESP32-S3/RS485_TX
- U6 pad 29: unconnected-(U6-IO36-Pad29) -> /ESP32-S3/DE
- U6 pad 30: unconnected-(U6-IO37-Pad30) -> /Circuito digital/DI0
- U6 pad 32: unconnected-(U6-IO39-Pad32) -> /Circuito Analógico/MCU-AO0
- U6 pad 33: unconnected-(U6-IO40-Pad33) -> /Circuito Analógico/MCU-AO1
- U6 pad 34: unconnected-(U6-IO41-Pad34) -> /Circuito digital/DI1
- U6 pad 35: unconnected-(U6-IO42-Pad35) -> /Circuito digital/DI2
- U6 pad 38: unconnected-(U6-IO2-Pad38) -> /Circuito Analógico/MCU-AI1
- U6 pad 39: unconnected-(U6-IO1-Pad39) -> /Circuito Analógico/MCU-AI0
- U6 pad 8: unconnected-(U6-IO15-Pad8) -> /Circuito digital/RELE 5
- U6 pad 9: unconnected-(U6-IO16-Pad9) -> /Circuito digital/RELE 6
- U9 pad 2: /~{RE} -> GND
- U9 pad 3: /DE -> GND
- U9 pad 4: /RS485_TX -> /Circuito digital/DI2
