File: Controlador-Compressor/Controlador-Compressor.kicad_sch (KiCad schematic)
At the start: 120 parts, among them J1 RELÉ-1, J10 USB_C_Receptacle, J2 RELÉ-2, J3 RELÉ-3, J4 RELÉ-4, J5 RELÉ-5, J6 Alimentação, J9 Analogico, J9 USB_C_Receptacle, J9 modbus, K1 FINDER-36.11, K2 FINDER-36.11, K3 FINDER-36.11, K4 FINDER-36.11, K5 FINDER-36.11, Q1 BC817, Q2 BC817, SW1 BOOT0, SW2 RST, U1 ESP32S3WROOM1N8R8, U1 PC817, U10 CP2102N-Axx-xQFN28, U2 PC817, U3 PC817, U4 PC817, U5 PC817, U6 LM358, U7 AMS1117-3.3, U9 SN75176ADR

Commit message: mei caminho andado
Parts:
- removed C1 (x2), C3: 10uF, Capacitor_SMD:C_0603_1608Metric_Pad1.08x0.95mm_HandSolder, symbol Industronic_v_0.1-rescue:C_Small-Device
- removed C10, C12, C13, C19, C21, C22: 220nF, Capacitor_SMD:C_0402_1005Metric, symbol Device:C_Small
- removed C11, C18, C20, C9: 1.5pF, Capacitor_SMD:C_0402_1005Metric, symbol Device:C
- removed C14, C15, C23, C24: 10uF, Capacitor_SMD:C_0603_1608Metric, symbol Device:C_Polarized_Small_US
- removed C17, C25, C7: 1uF, symbol Device:C
- removed C2: 1uF, Capacitor_SMD:C_0603_1608Metric_Pad1.08x0.95mm_HandSolder, symbol Industronic_v_0.1-rescue:C_Small-Device
- removed C26, C6: 10uF, symbol Device:C
- removed C4, C5, C8: 100nF, symbol Device:C
- removed D1, D2, D3, D4, D5: D, Diode_THT:D_A-405_P2.54mm_Vertical_KathodeUp, symbol Device:D
- removed D10, D6, D7, D8, D9: LED, LED_SMD:LED_0805_2012Metric_Pad1.15x1.40mm_HandSolder, symbol Device:LED
- removed D11, D12: SMCJ7,0CA, symbol Device:D_Zener_Small_Filled
- removed D13: WS2812B, LED_SMD:LED_WS2812B_PLCC4_5.0x5.0mm_P3.2mm, symbol LED:WS2812B
- removed D14, D16: SRV05-4-P-T7, Package_TO_SOT_SMD:SOT-23-6, symbol dk_TVS-Diodes:IP4220CZ6_125
- removed D15, D17, D18: 1N5819H2-7-F, symbol Device:D_Small_Filled
- removed F1, F2, F3, F4: 0ZRE0008FF1C, symbol Device:Polyfuse_Small
- removed FL1, FL2: ECMF02, Package_DFN_QFN:ST_UQFN-6L_1.5x1.7mm_Pitch0.5mm, symbol esteban2:ECMF02
- removed IN+1: IN+, Connector_PinHeader_2.54mm:PinHeader_1x01_P2.54mm_Vertical, symbol Connector_Generic:Conn_01x01
- removed IN-1: IN-, Connector_PinHeader_2.54mm:PinHeader_1x01_P2.54mm_Vertical, symbol Connector_Generic:Conn_01x01
- removed J1: RELÉ-1, Connector_Phoenix_MSTB:PhoenixContact_MSTBA_2,5_3-G-5,08_1x03_P5.08mm_Horizontal, symbol Connector_Generic:Conn_01x03
- removed J10, J9: USB_C_Receptacle, usb-c:usb-eps, symbol Connector:USB_C_Receptacle
- removed J2: RELÉ-2, Connector_Phoenix_MSTB:PhoenixContact_MSTBA_2,5_3-G-5,08_1x03_P5.08mm_Horizontal, symbol Connector_Generic:Conn_01x03
- removed J3: RELÉ-3, Connector_Phoenix_MSTB:PhoenixContact_MSTBA_2,5_3-G-5,08_1x03_P5.08mm_Horizontal, symbol Connector_Generic:Conn_01x03
- removed J4: RELÉ-4, Connector_Phoenix_MSTB:PhoenixContact_MSTBA_2,5_3-G-5,08_1x03_P5.08mm_Horizontal, symbol Connector_Generic:Conn_01x03
- removed J5: RELÉ-5, Connector_Phoenix_MSTB:PhoenixContact_MSTBA_2,5_3-G-5,08_1x03_P5.08mm_Horizontal, symbol Connector_Generic:Conn_01x03
- removed J9: Analogico, Connector_Phoenix_MSTB:PhoenixContact_MSTBA_2,5_3-G-5,08_1x03_P5.08mm_Horizontal, symbol Connector_Generic:Conn_01x03
- removed J9: modbus, Connector_Phoenix_MSTB:PhoenixContact_MSTBA_2,5_3-G-5,08_1x03_P5.08mm_Horizontal, symbol Connector_Generic:Conn_01x03
- removed JP1: GPIO3, symbol Jumper:SolderJumper_3_Open
- removed K1, K2, K3, K4, K5: FINDER-36.11, Relay_THT:Relay_SPDT_Finder_36.11, symbol Relay:FINDER-36.11
- removed L1, L2: FBMJ2125HS420-T, Inductor_SMD:L_0805_2012Metric, symbol Device:L_Ferrite
- removed OUT+1: OUT+, Connector_PinHeader_2.54mm:PinHeader_1x01_P2.54mm_Vertical, symbol Connector_Generic:Conn_01x01
- removed OUT-1: OUT-, Connector_PinHeader_2.54mm:PinHeader_1x01_P2.54mm_Vertical, symbol Connector_Generic:Conn_01x01
- removed Q1, Q2: BC817, Package_TO_SOT_SMD:SOT-23, symbol Transistor_BJT:BC817
- removed R1, R2, R3, R4, R5: 1k, Resistor_SMD:R_0603_1608Metric_Pad0.98x0.95mm_HandSolder, symbol Device:R
- removed R10, R11, R12, R13, R14, R15, R20, R25, R26: 10k, symbol Device:R
- removed R16, R17, R27, R28: 100k, Resistor_SMD:R_0402_1005Metric, symbol Device:R
- removed R18, R19, R29, R30: 5.1K, Resistor_SMD:R_0402_1005Metric, symbol Device:R_Small
- removed R21, R22: 0R, symbol Device:R
- removed R23: 22.1k, symbol Device:R
- removed R24: 47.5k, symbol Device:R
- removed R6, R7: 3.3k, Resistor_SMD:R_0805_2012Metric_Pad1.20x1.40mm_HandSolder, symbol Device:R
- removed R6 (x2): 33k, Resistor_SMD:R_0805_2012Metric_Pad1.20x1.40mm_HandSolder, symbol Device:R
- removed R8 (x2): 100k, Resistor_SMD:R_0805_2012Metric_Pad1.20x1.40mm_HandSolder, symbol Device:R
- removed R8, R9: 10k, Resistor_SMD:R_0805_2012Metric_Pad1.20x1.40mm_HandSolder, symbol Device:R
- removed SW1: BOOT0, symbol Switch:SW_MEC_5E
- removed SW2: RST, symbol Switch:SW_MEC_5E
- removed U1: ESP32S3WROOM1N8R8, esp32s3:XCVR_ESP32S3WROOM1N8R8, symbol Esp32S3:ESP32S3WROOM1N8R8
- removed U1, U2, U3, U4, U5: PC817, Package_DIP:DIP-4_W7.62mm, symbol Isolator:PC817
- removed U10: CP2102N-Axx-xQFN28, Package_DFN_QFN:QFN-28-1EP_5x5mm_P0.5mm_EP3.35x3.35mm, symbol Interface_USB:CP2102N-Axx-xQFN28
- removed U6: LM358, Package_DIP:DIP-8_W7.62mm, symbol Amplifier_Operational:LM358
- removed U7: AMS1117-3.3, Package_TO_SOT_SMD:SOT-223-3_TabPin2, symbol Regulator_Linear:AMS1117-3.3
- removed U9: SN75176ADR, Package_SO:SOIC-8_3.9x4.9mm_P1.27mm, symbol Interface_UART:SN75176AD
- added J1: RELÉ 2, Connector_Phoenix_MSTB:PhoenixContact_MSTBA_2,5_2-G-5,08_1x02_P5.08mm_Horizontal, symbol Connector_Generic:Conn_01x02
- added J11: RELÉ 7, Connector_Phoenix_MSTB:PhoenixContact_MSTBA_2,5_2-G-5,08_1x02_P5.08mm_Horizontal, symbol Connector_Generic:Conn_01x02
- added J12: DB9 - ModBus shield, symbol Connector:DE9_Plug
- added J13: AI0 ... AI11, Connector_Phoenix_MSTB:PhoenixContact_MSTBA_2,5_12-G-5,08_1x12_P5.08mm_Horizontal, symbol Connector_Generic:Conn_01x12
- added J14: AO0 ... AO3, Connector_Phoenix_MSTB:PhoenixContact_MSTBA_2,5_4-G-5,08_1x04_P5.08mm_Horizontal, symbol Connector_Generic:Conn_01x04
- added J15: RELÉ 8, Connector_Phoenix_MSTB:PhoenixContact_MSTBA_2,5_2-G-5,08_1x02_P5.08mm_Horizontal, symbol Connector_Generic:Conn_01x02
- added J2: RELÉ 1, Connector_Phoenix_MSTB:PhoenixContact_MSTBA_2,5_2-G-5,08_1x02_P5.08mm_Horizontal, symbol Connector_Generic:Conn_01x02
- added J3: RELÉ 3, Connector_Phoenix_MSTB:PhoenixContact_MSTBA_2,5_2-G-5,08_1x02_P5.08mm_Horizontal, symbol Connector_Generic:Conn_01x02
- added J4: RELÉ 4, Connector_Phoenix_MSTB:PhoenixContact_MSTBA_2,5_2-G-5,08_1x02_P5.08mm_Horizontal, symbol Connector_Generic:Conn_01x02
- added J5: RELÉ 5, Connector_Phoenix_MSTB:PhoenixContact_MSTBA_2,5_2-G-5,08_1x02_P5.08mm_Horizontal, symbol Connector_Generic:Conn_01x02
- added J8: RELÉ 6, Connector_Phoenix_MSTB:PhoenixContact_MSTBA_2,5_2-G-5,08_1x02_P5.08mm_Horizontal, symbol Connector_Generic:Conn_01x02
Connections:
- net +24V: now also J12.7
- net +5V: now also J12.6
- new net 24V-Return: J12.2
- new net 5V-Return: J12.5
- new net Analógico/AI0: J13.1 (Pin_1)
- new net Analógico/AI1: J13.2 (Pin_2)
- new net Analógico/AI10: J13.11 (Pin_11)
- new net Analógico/AI11: J13.12 (Pin_12)
- new net Analógico/AI2: J13.3 (Pin_3)
- new net Analógico/AI3: J13.4 (Pin_4)
- new net Analógico/AI4: J13.5 (Pin_5)
- new net Analógico/AI5: J13.6 (Pin_6)
- new net Analógico/AI6: J13.7 (Pin_7)
- new net Analógico/AI7: J13.8 (Pin_8)
- new net Analógico/AI8: J13.9 (Pin_9)
- new net Analógico/AI9: J13.10 (Pin_10)
- new net Analógico/AO1: J14.2 (Pin_2)
- new net Analógico/AO2: J14.3 (Pin_3)
- new net Analógico/AO3: J14.4 (Pin_4)
- new net MODBUS-RTS: J12.4
- new net MODBUS-SHIELD: J12.1
- new net Modbus/A: J12.8
- new net Modbus/B: J12.3
- new net Potência/COM0: J2.2 (Pin_2)
- new net Potência/COM1: J1.2 (Pin_2)
- new net Potência/COM2: J3.2 (Pin_2)
- new net Potência/COM3: J4.2 (Pin_2)
- new net Potência/COM4: J5.2 (Pin_2)
- new net Potência/COM5: J8.2 (Pin_2)
- new net Potência/COM6: J11.2 (Pin_2)
- new net Potência/COM7: J15.2 (Pin_2)
- new net Potência/DO0: J2.1 (Pin_1)
- new net Potência/DO1: J1.1 (Pin_1)
- new net Potência/DO2: J3.1 (Pin_1)
- new net Potência/DO3: J4.1 (Pin_1)
- new net Potência/DO4: J5.1 (Pin_1)
- new net Potência/DO5: J8.1 (Pin_1)
- new net Potência/DO6: J11.1 (Pin_1)
- new net Potência/DO7: J15.1 (Pin_1)
- no-connect marks 40 -> 1
Other:
- added sheet Analógico (Analógico.kicad_sch)
- added sheet ESP32-S3 (ESP32-S3.kicad_sch)
- added sheet Fonte-Placa (Fonte-Placa.kicad_sch)
- added sheet Modbus (Modbus.kicad_sch)
- added sheet Potência (Potência.kicad_sch)
- added sheet USB->OTG (USB->OTG.kicad_sch)
- added sheet USB->UART (USB->UART.kicad_sch)
- note added: "0V -> 10V"
- note added: "RS485 MODBUS pinout Siemens: https://support.industry.siemens.com/forum/br/en/posts/rs485-pin-out-details-of-port-in-cpu-226/160925"
- note removed: "Analog outputs"
- note removed: "ESP32-S3-DualCore-240MHz"
- note removed: "Fonte"
- note removed: "GANHO ~4"
- note removed: "POWER SUPPLY"
- note removed: "RGB"
- note removed: "RS485 - Modbus"
- note removed: "Relés"
- note removed: "USB -> UART"
- note removed: "USB TO ESP"
- note removed: "USB to UART"

Commit message: terminei escopo do projeto
Parts:
- removed J1: RELÉ 2, Connector_Phoenix_MSTB:PhoenixContact_MSTBA_2,5_2-G-5,08_1x02_P5.08mm_Horizontal, symbol Connector_Generic:Conn_01x02
- removed J11: RELÉ 7, Connector_Phoenix_MSTB:PhoenixContact_MSTBA_2,5_2-G-5,08_1x02_P5.08mm_Horizontal, symbol Connector_Generic:Conn_01x02
- removed J13: AI0 ... AI11, Connector_Phoenix_MSTB:PhoenixContact_MSTBA_2,5_12-G-5,08_1x12_P5.08mm_Horizontal, symbol Connector_Generic:Conn_01x12
- removed J14: AO0 ... AO3, Connector_Phoenix_MSTB:PhoenixContact_MSTBA_2,5_4-G-5,08_1x04_P5.08mm_Horizontal, symbol Connector_Generic:Conn_01x04
- removed J15: RELÉ 8, Connector_Phoenix_MSTB:PhoenixContact_MSTBA_2,5_2-G-5,08_1x02_P5.08mm_Horizontal, symbol Connector_Generic:Conn_01x02
- removed J2: RELÉ 1, Connector_Phoenix_MSTB:PhoenixContact_MSTBA_2,5_2-G-5,08_1x02_P5.08mm_Horizontal, symbol Connector_Generic:Conn_01x02
- removed J3: RELÉ 3, Connector_Phoenix_MSTB:PhoenixContact_MSTBA_2,5_2-G-5,08_1x02_P5.08mm_Horizontal, symbol Connector_Generic:Conn_01x02
- removed J4: RELÉ 4, Connector_Phoenix_MSTB:PhoenixContact_MSTBA_2,5_2-G-5,08_1x02_P5.08mm_Horizontal, symbol Connector_Generic:Conn_01x02
- removed J5: RELÉ 5, Connector_Phoenix_MSTB:PhoenixContact_MSTBA_2,5_2-G-5,08_1x02_P5.08mm_Horizontal, symbol Connector_Generic:Conn_01x02
- removed J8: RELÉ 6, Connector_Phoenix_MSTB:PhoenixContact_MSTBA_2,5_2-G-5,08_1x02_P5.08mm_Horizontal, symbol Connector_Generic:Conn_01x02
- added J1: Entradas Digitais, symbol Connector_Generic:Conn_01x05
- added J11: Saídas Relé, Connector_Phoenix_MSTB:PhoenixContact_MSTBA_2,5_12-G-5,08_1x12_P5.08mm_Horizontal, symbol Connector_Generic:Conn_01x12
- added J13: Analógico, Connector_Phoenix_MSTB:PhoenixContact_MSTBA_2,5_16-G-5,08_1x16_P5.08mm_Horizontal, symbol Connector_Generic:Conn_01x16
- added J16: Nextion, Connector_JST:JST_EH_B4B-EH-A_1x04_P2.50mm_Vertical, symbol Connector_Generic:Conn_01x04
Connections:
- net +5V: now also J16.1 (Pin_1)
- net Circuito Analógico/AI0: now also J13.5 (Pin_5)
- net Circuito Analógico/AI1: now also J13.6 (Pin_6)
- net Circuito Analógico/AI10: now also J13.15 (Pin_15)
- net Circuito Analógico/AI11: now also J13.16 (Pin_16)
- net Circuito Analógico/AI2: now also J13.7 (Pin_7)
- net Circuito Analógico/AI3: now also J13.8 (Pin_8)
- net Circuito Analógico/AI4: now also J13.9 (Pin_9)
- net Circuito Analógico/AI5: now also J13.10 (Pin_10)
- net Circuito Analógico/AI6: now also J13.11 (Pin_11)
- net Circuito Analógico/AI7: now also J13.12 (Pin_12)
- net Circuito Analógico/AI8: now also J13.13 (Pin_13)
- net Circuito Analógico/AI9: now also J13.14 (Pin_14)
- net Circuito Analógico/AO0: now also J13.1 (Pin_1)
- net Circuito Analógico/AO1: now also J13.2 (Pin_2)
- net Circuito Analógico/AO2: now also J13.3 (Pin_3)
- net Circuito Analógico/AO3: now also J13.4 (Pin_4)
- net GND: now also J16.4 (Pin_4)
- net Circuito digital/COM0: now also J11.2 (Pin_2)
- net Circuito digital/COM1: now also J11.4 (Pin_4)
- net Circuito digital/COM2: now also J11.6 (Pin_6)
- net Circuito digital/COM3: now also J11.8 (Pin_8)
- net Circuito digital/COM4: now also J11.10 (Pin_10)
- net Circuito digital/COM5: now also J11.12 (Pin_12)
- net Circuito digital/DO0: now also J11.1 (Pin_1)
- net Circuito digital/DO1: now also J11.3 (Pin_3)
- net Circuito digital/DO2: now also J11.5 (Pin_5)
- net Circuito digital/DO3: now also J11.7 (Pin_7)
- net Circuito digital/DO4: now also J11.9 (Pin_9)
- net Circuito digital/DO5: now also J11.11 (Pin_11)
- new net Circuito digital/DI0-24V: J1.1 (Pin_1)
- new net Circuito digital/DI1-24V: J1.2 (Pin_2)
- new net Circuito digital/DI2-24V: J1.3 (Pin_3)
- new net Circuito digital/DI3-24V: J1.4 (Pin_4)
- new net Circuito digital/DI4-24V: J1.5 (Pin_5)
- new net ESP32-S3/RX-Nextion: J16.2 (Pin_2)
- new net ESP32-S3/Tx-Nextion: J16.3 (Pin_3)
Other:
- sheet Analógico renamed Circuito Analógico
- sheet Potência renamed Circuito digital
- sheet Circuito digital ports: added DI0, DI0-24V, DI1, DI1-24V, DI2, DI2-24V, DI3, DI3-24V, DI4, DI4-24V; removed COM6, COM7, DO6, DO7, RELE 7, RELE 8
- sheet ESP32-S3 ports: added DI0, DI1, DI2, DI3, DI4, GPIO0, OTG-D+, OTG-D-, RST, RX-Nextion, RXD0, TXD0, Tx-Nextion; removed MCU-AI10, MCU-AI11, MCU-AO2, MCU-AO3, RELE 7, RELE 8
- note added: "10 entradas analógicas"
- note added: "2 saídas analogicas"
- note added: "5 entradas Digitais"
- note added: "6 Saídas Digitais"
- note added: "IHM"
- note added: "RS-485 MODBUS"
- note added: "Todas saidas Normalmente Abertas COM0 __/ __ DO0"
- note added: "USB OTG"
- note added: "USB SERIAL"
- moved on the sheet: J6
