File: Controlador-Compressor/ESP32-S3.kicad_sch (KiCad schematic)
At the start: 16 parts, among them SW1 BOOT0, SW2 RST, U1 ESP32S3WROOM1N8R8

Commit message: terminei escopo do projeto
Connections:
- net GPIO3 is gone; now on net MCU-AI2: JP1.2 (C)
- net MCU-AI10 is gone; now on net RELE 1: U1.19 (IO11)
- net MCU-AI11 is gone; now on net RELE 2: U1.20 (IO12)
- net RELE 1: no longer U1.22 (IO14)
- net RELE 2: no longer U1.8 (IO15)
- net RELE 3: now also U1.21 (IO13); no longer U1.9 (IO16)
- net RELE 4: now also U1.22 (IO14); no longer U1.10 (IO17)
- net RELE 5: now also U1.8 (IO15); no longer U1.11 (IO18)
- net RELE 6: now also U1.9 (IO16); no longer U1.30 (IO37)
- net GPIO19 renamed OTG-D-
- net GPIO20 renamed OTG-D+
- net MCU-AO2 renamed DI1
- net MCU-AO3 renamed DI2
- net RELE 7 renamed DI3
- net RELE 8 renamed DI4
- new net DI0: U1.30 (IO37)
- new net RX-Nextion: U1.10 (IO17)
- new net Tx-Nextion: U1.11 (IO18)
Other:
- company: (none) -> Linear Compressores
- title: (none) -> Controlador Compressor
- moved on the sheet: C4, C5, C6, C7, C8, D13, JP1, R10, R11, R12, R13, R14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
