File: Controlador-Compressor/Modbus.kicad_sch (KiCad schematic)
At the start: 6 parts

Commit message: terminei escopo do projeto
Other:
- company: (none) -> Linear Compressores
- title: (none) -> Controlador Compressor
Changed lines of the file:
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@@
 (kicad_sch (version 20230121) (generator eeschema)
   (paper "A4")
+  (title_block
+    (title "Controlador Compressor")
+    (date "2023-03-07")
+    (rev "1")
+    (company "Linear Compressores")
+    (comment 1 "Autor: Ícaro Fernando")
+  )
   (junction (at 131.445 75.565) (diameter 0) (color 0 0 0 0)
   )
