File: Controlador-Compressor/Potência.kicad_sch (KiCad schematic)
At the start: 48 parts, among them K1 FINDER-36.11, K2 FINDER-36.11, Q3 BC817

Commit message: terminei escopo do projeto
Parts:
- removed D1 (x2): D, Diode_THT:D_A-405_P2.54mm_Vertical_KathodeUp, symbol Device:D
- removed D6 (x2): LED, LED_SMD:LED_0805_2012Metric_Pad1.15x1.40mm_HandSolder, symbol Device:LED
- removed K1 (x2): FINDER-36.11, Relay_THT:Relay_SPDT_Finder_36.11, symbol Relay:FINDER-36.11
- removed Q3 (x2): BC817, Package_TO_SOT_SMD:SOT-23, symbol Transistor_BJT:BC817
- removed R1 (x4): 1k, Resistor_SMD:R_0603_1608Metric_Pad0.98x0.95mm_HandSolder, symbol Device:R
- added D13, D23, D24, D25, D26: LED, symbol Device:LED
- added R45, R46, R47, R48, R49, R50, R51, R52, R53, R54: R, symbol Device:R
- added U10, U11, U4, U5, U9: PC817, Package_DIP:DIP-4_W7.62mm, symbol Isolator:PC817
Connections:
- net GND: now also U10.2, U10.3, U11.2, U11.3, U4.2, U4.3, U5.2, U5.3, U9.2, U9.3
- new net: D23.1 (K), R45.2
- new net: R52.1, U10.1
- new net: D25.1 (K), R52.2
- new net: R48.1, U5.1
- new net: R50.1, U9.1
- new net: D24.1 (K), R50.2
- new net: D13.1 (K), R48.2
- new net: R45.1, U4.1
- new net: R54.1, U11.1
- new net: D26.1 (K), R54.2
- new net +3.3V: R46.1, R47.1, R49.1, R51.1, R53.1
- new net DI0: R46.2, U4.4
- new net DI0-24V: D23.2 (A)
- new net DI1: R47.2, U5.4
- new net DI1-24V: D13.2 (A)
- new net DI2: R49.2, U9.4
- new net DI2-24V: D24.2 (A)
- new net DI3: R51.2, U10.4
- new net DI3-24V: D25.2 (A)
- new net DI4: R53.2, U11.4
- new net DI4-24V: D26.2 (A)
Other:
- note added: "Saídas Relés"
- note removed: "Relés"
- company: (none) -> Linear Compressores
- title: (none) -> Controlador Compressor
- moved on the sheet: D1, D2, D6, K1, K2, Q3, R1
