File: Controlador-Compressor/USB->OTG.kicad_sch (KiCad schematic)
At the start: 16 parts, among them J10 USB_C_Receptacle

Commit message: terminei escopo do projeto
Other:
- company: (none) -> Linear Compressores
- title: (none) -> Controlador Compressor
Changed lines of the file:
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@@
 (kicad_sch (version 20230121) (generator eeschema)
   (paper "A4")
+  (title_block
+    (title "Controlador Compressor")
+    (date "2023-03-07")
+    (rev "1")
+    (company "Linear Compressores")
+    (comment 1 "Autor: Ícaro Fernando")
+  )
   (junction (at 133.35 102.87) (diameter 0) (color 0 0 0 0)
   )
@@
     (stroke (width 0) (type default))
   )
-  (wire (pts (xy 109.22 59.69) (xy 116.84 59.69))
+  (wire (pts (xy 104.14 59.69) (xy 116.84 59.69))
     (stroke (width 0) (type default))
   )
@@
     (stroke (width 0) (type default))
   )
-  (wire (pts (xy 89.535 55.88) (xy 97.155 55.88))
+  (wire (pts (xy 89.535 55.88) (xy 97.79 55.88))
     (stroke (width 0) (type default))
   )
@@
     (effects (font (size 1.27 1.27)) (justify right bottom))
   )
-  (label "ESP_D-" (at 97.155 55.88 180) (fields_autoplaced)
+  (label "ESP_D-" (at 97.79 55.88 180) (fields_autoplaced)
     (effects (font (size 1.27 1.27)) (justify right bottom))
   )
@@
     (effects (font (size 1.27 1.27)) (justify right bottom))
   )
-  (label "ESP_SHIELD" (at 109.22 59.69 0) (fields_autoplaced)
+  (label "ESP_SHIELD" (at 104.14 59.69 0) (fields_autoplaced)
     (effects (font (size 1.27 1.27)) (justify left bottom))
   )
@@
           (reference "#PWR040") (unit 1)
         )
-        (path "/804a4dd1-72d2-453c-88d6-2d38d7bf9060/4780c35f-b56d-4192-ad95-c1302f9dbd7c"
+        (path "/804a4dd1-72d2-453c-88d6-2d38d7bf9060/a41eed78-77a0-4dcd-8138-22abfedc3c2b"
           (reference "#PWR040") (unit 1)
         )
@@
           (reference "C5") (unit 1)
         )
-        (path "/804a4dd1-72d2-453c-88d6-2d38d7bf9060/4780c35f-b56d-4192-ad95-c1302f9dbd7c"
+        (path "/804a4dd1-72d2-453c-88d6-2d38d7bf9060/a41eed78-77a0-4dcd-8138-22abfedc3c2b"
           (reference "C5") (unit 1)
         )
@@
           (reference "#PWR038") (unit 1)
         )
-        (path "/804a4dd1-72d2-453c-88d6-2d38d7bf9060/4780c35f-b56d-4192-ad95-c1302f9dbd7c"
+        (path "/804a4dd1-72d2-453c-88d6-2d38d7bf9060/a41eed78-77a0-4dcd-8138-22abfedc3c2b"
           (reference "#PWR038") (unit 1)
         )
@@
           (reference "C17") (unit 1)
         )
-        (path "/804a4dd1-72d2-453c-88d6-2d38d7bf9060/4780c35f-b56d-4192-ad95-c1302f9dbd7c"
+        (path "/804a4dd1-72d2-453c-88d6-2d38d7bf9060/a41eed78-77a0-4dcd-8138-22abfedc3c2b"
           (reference "C17") (unit 1)
         )
@@
           (reference "L2") (unit 1)
         )
-        (path "/804a4dd1-72d2-453c-88d6-2d38d7bf9060/4780c35f-b56d-4192-ad95-c1302f9dbd7c"
+        (path "/804a4dd1-72d2-453c-88d6-2d38d7bf9060/a41eed78-77a0-4dcd-8138-22abfedc3c2b"
           (reference "L2") (unit 1)
         )
@@
           (reference "#PWR062") (unit 1)
         )
-        (path "/804a4dd1-72d2-453c-88d6-2d38d7bf9060/4780c35f-b56d-4192-ad95-c1302f9dbd7c"
+        (path "/804a4dd1-72d2-453c-88d6-2d38d7bf9060/a41eed78-77a0-4dcd-8138-22abfedc3c2b"
           (reference "#PWR062") (unit 1)
         )
@@
           (reference "C15") (unit 1)
         )
-        (path "/804a4dd1-72d2-453c-88d6-2d38d7bf9060/4780c35f-b56d-4192-ad95-c1302f9dbd7c"
+        (path "/804a4dd1-72d2-453c-88d6-2d38d7bf9060/a41eed78-77a0-4dcd-8138-22abfedc3c2b"
           (reference "C15") (unit 1)
         )
@@
           (reference "#PWR033") (unit 1)
         )
-        (path "/804a4dd1-72d2-453c-88d6-2d38d7bf9060/4780c35f-b56d-4192-ad95-c1302f9dbd7c"
+        (path "/804a4dd1-72d2-453c-88d6-2d38d7bf9060/a41eed78-77a0-4dcd-8138-22abfedc3c2b"
           (reference "#PWR033") (unit 1)
         )
@@
           (reference "C13") (unit 1)
         )
-        (path "/804a4dd1-72d2-453c-88d6-2d38d7bf9060/4780c35f-b56d-4192-ad95-c1302f9dbd7c"
+        (path "/804a4dd1-72d2-453c-88d6-2d38d7bf9060/a41eed78-77a0-4dcd-8138-22abfedc3c2b"
           (reference "C13") (unit 1)
         )
@@
           (reference "R14") (unit 1)
         )
-        (path "/804a4dd1-72d2-453c-88d6-2d38d7bf9060/4780c35f-b56d-4192-ad95-c1302f9dbd7c"
+        (path "/804a4dd1-72d2-453c-88d6-2d38d7bf9060/a41eed78-77a0-4dcd-8138-22abfedc3c2b"
           (reference "R14") (unit 1)
         )
@@
           (reference "C11") (unit 1)
         )
-        (path "/804a4dd1-72d2-453c-88d6-2d38d7bf9060/4780c35f-b56d-4192-ad95-c1302f9dbd7c"
+        (path "/804a4dd1-72d2-453c-88d6-2d38d7bf9060/a41eed78-77a0-4dcd-8138-22abfedc3c2b"
           (reference "C11") (unit 1)
         )
@@
           (reference "#PWR036") (unit 1)
         )
-        (path "/804a4dd1-72d2-453c-88d6-2d38d7bf9060/4780c35f-b56d-4192-ad95-c1302f9dbd7c"
+        (path "/804a4dd1-72d2-453c-88d6-2d38d7bf9060/a41eed78-77a0-4dcd-8138-22abfedc3c2b"
           (reference "#PWR036") (unit 1)
         )
@@
           (reference "C9") (unit 1)
         )
-        (path "/804a4dd1-72d2-453c-88d6-2d38d7bf9060/4780c35f-b56d-4192-ad95-c1302f9dbd7c"
+        (path "/804a4dd1-72d2-453c-88d6-2d38d7bf9060/a41eed78-77a0-4dcd-8138-22abfedc3c2b"
           (reference "C9") (unit 1)
         )
@@
           (reference "#PWR061") (unit 1)
         )
-        (path "/804a4dd1-72d2-453c-88d6-2d38d7bf9060/4780c35f-b56d-4192-ad95-c1302f9dbd7c"
+        (path "/804a4dd1-72d2-453c-88d6-2d38d7bf9060/a41eed78-77a0-4dcd-8138-22abfedc3c2b"
           (reference "#PWR061") (unit 1)
         )
@@
           (reference "R13") (unit 1)
         )
-        (path "/804a4dd1-72d2-453c-88d6-2d38d7bf9060/4780c35f-b56d-4192-ad95-c1302f9dbd7c"
+        (path "/804a4dd1-72d2-453c-88d6-2d38d7bf9060/a41eed78-77a0-4dcd-8138-22abfedc3c2b"
           (reference "R13") (unit 1)
         )
@@
           (reference "R16") (unit 1)
         )
-        (path "/804a4dd1-72d2-453c-88d6-2d38d7bf9060/4780c35f-b56d-4192-ad95-c1302f9dbd7c"
+        (path "/804a4dd1-72d2-453c-88d6-2d38d7bf9060/a41eed78-77a0-4dcd-8138-22abfedc3c2b"
           (reference "R16") (unit 1)
         )
@@
           (reference "#PWR057") (unit 1)
         )
-        (path "/804a4dd1-72d2-453c-88d6-2d38d7bf9060/4780c35f-b56d-4192-ad95-c1302f9dbd7c"
+        (path "/804a4dd1-72d2-453c-88d6-2d38d7bf9060/a41eed78-77a0-4dcd-8138-22abfedc3c2b"
           (reference "#PWR057") (unit 1)
         )
@@
           (reference "#PWR052") (unit 1)
         )
-        (path "/804a4dd1-72d2-453c-88d6-2d38d7bf9060/4780c35f-b56d-4192-ad95-c1302f9dbd7c"
+        (path "/804a4dd1-72d2-453c-88d6-2d38d7bf9060/a41eed78-77a0-4dcd-8138-22abfedc3c2b"
           (reference "#PWR052") (unit 1)
         )
@@
           (reference "#PWR060") (unit 1)
         )
-        (path "/804a4dd1-72d2-453c-88d6-2d38d7bf9060/4780c35f-b56d-4192-ad95-c1302f9dbd7c"
+        (path "/804a4dd1-72d2-453c-88d6-2d38d7bf9060/a41eed78-77a0-4dcd-8138-22abfedc3c2b"
           (reference "#PWR060") (unit 1)
         )
@@
           (reference "#PWR065") (unit 1)
         )
-        (path "/804a4dd1-72d2-453c-88d6-2d38d7bf9060/4780c35f-b56d-4192-ad95-c1302f9dbd7c"
+        (path "/804a4dd1-72d2-453c-88d6-2d38d7bf9060/a41eed78-77a0-4dcd-8138-22abfedc3c2b"
           (reference "#PWR065") (unit 1)
         )
@@
           (reference "D14") (unit 1)
         )
-        (path "/804a4dd1-72d2-453c-88d6-2d38d7bf9060/4780c35f-b56d-4192-ad95-c1302f9dbd7c"
+        (path "/804a4dd1-72d2-453c-88d6-2d38d7bf9060/a41eed78-77a0-4dcd-8138-22abfedc3c2b"
           (reference "D14") (unit 1)
         )
@@
           (reference "D17") (unit 1)
         )
-        (path "/804a4dd1-72d2-453c-88d6-2d38d7bf9060/4780c35f-b56d-4192-ad95-c1302f9dbd7c"
+        (path "/804a4dd1-72d2-453c-88d6-2d38d7bf9060/a41eed78-77a0-4dcd-8138-22abfedc3c2b"
           (reference "D17") (unit 1)
         )
@@
           (reference "R11") (unit 1)
         )
-        (path "/804a4dd1-72d2-453c-88d6-2d38d7bf9060/4780c35f-b56d-4192-ad95-c1302f9dbd7c"
+        (path "/804a4dd1-72d2-453c-88d6-2d38d7bf9060/a41eed78-77a0-4dcd-8138-22abfedc3c2b"
           (reference "R11") (unit 1)
         )
@@
           (reference "C7") (unit 1)
         )
-        (path "/804a4dd1-72d2-453c-88d6-2d38d7bf9060/4780c35f-b56d-4192-ad95-c1302f9dbd7c"
+        (path "/804a4dd1-72d2-453c-88d6-2d38d7bf9060/a41eed78-77a0-4dcd-8138-22abfedc3c2b"
           (reference "C7") (unit 1)
         )
@@
           (reference "#PWR043") (unit 1)
         )
-        (path "/804a4dd1-72d2-453c-88d6-2d38d7bf9060/4780c35f-b56d-4192-ad95-c1302f9dbd7c"
+        (path "/804a4dd1-72d2-453c-88d6-2d38d7bf9060/a41eed78-77a0-4dcd-8138-22abfedc3c2b"
           (reference "#PWR043") (unit 1)
         )
@@
           (reference "J10") (unit 1)
         )
-        (path "/804a4dd1-72d2-453c-88d6-2d38d7bf9060/4780c35f-b56d-4192-ad95-c1302f9dbd7c"
+        (path "/804a4dd1-72d2-453c-88d6-2d38d7bf9060/a41eed78-77a0-4dcd-8138-22abfedc3c2b"
           (reference "J10") (unit 1)
         )
@@
           (reference "#PWR041") (unit 1)
         )
-        (path "/804a4dd1-72d2-453c-88d6-2d38d7bf9060/4780c35f-b56d-4192-ad95-c1302f9dbd7c"
+        (path "/804a4dd1-72d2-453c-88d6-2d38d7bf9060/a41eed78-77a0-4dcd-8138-22abfedc3c2b"
           (reference "#PWR041") (unit 1)
         )
@@
           (reference "#PWR054") (unit 1)
         )
-        (path "/804a4dd1-72d2-453c-88d6-2d38d7bf9060/4780c35f-b56d-4192-ad95-c1302f9dbd7c"
+        (path "/804a4dd1-72d2-453c-88d6-2d38d7bf9060/a41eed78-77a0-4dcd-8138-22abfedc3c2b"
           (reference "#PWR054") (unit 1)
         )
@@
           (reference "FL2") (unit 1)
         )
-        (path "/804a4dd1-72d2-453c-88d6-2d38d7bf9060/4780c35f-b56d-4192-ad95-c1302f9dbd7c"
+        (path "/804a4dd1-72d2-453c-88d6-2d38d7bf9060/a41eed78-77a0-4dcd-8138-22abfedc3c2b"
           (reference "FL2") (unit 1)
         )
