File: Controlador-Compressor/USB->UART.kicad_sch (KiCad schematic)
At the start: 29 parts, among them J9 USB_C_Receptacle, Q1 BC817, Q2 BC817, U10 CP2102N-Axx-xQFN28

Commit message: terminei escopo do projeto
Other:
- company: (none) -> Linear Compressores
- title: (none) -> Controlador Compressor
